Commit message: Imported upstream version '6.0.0' of 'upstream'

File: exotica_examples/resources/robots/quadrotor.urdf (robot description, URDF)
Before this commit: robot quadrotor, 1 links, 0 joints
Links:
- added link base_inertial, mass 1.477
- link base_link: mass 1.477 -> None
Joints:
- added joint base_to_inertia: type fixed, parent base_link, child base_inertial

File: exotica_examples/resources/robots/valkyrie_sim.urdf (robot description, URDF)
Before this commit: robot valkyrie, 84 links, 83 joints
Links:
- link head_imu_link: geometry 
- link l_hand_force_torque: geometry 
- link left_palm: geometry 
- link r_hand_force_torque: geometry 
- link right_palm: geometry 

File: exotica_examples/test/resources/mesh_vs_mesh_distance.urdf (robot description, URDF)
Before this commit: robot A_vs_B, 2 links, 1 joints
Links:
- link A: geometry collision mesh filename=package://exotica_examples/test/resources/cube.obj; visual mesh filename=package://exotica_examples/test/resources/cube.obj
- link B: geometry collision mesh filename=package://exotica_examples/test/resources/uvsphere.obj; visual mesh filename=package://exotica_examples/test/resources/uvsphere.obj

File: exotica_examples/test/resources/mesh_vs_mesh_penetrating.urdf (robot description, URDF)
Before this commit: robot A_vs_B, 2 links, 1 joints
Links:
- link A: geometry collision mesh filename=package://exotica_examples/test/resources/cube.obj; visual mesh filename=package://exotica_examples/test/resources/cube.obj
- link B: geometry collision mesh filename=package://exotica_examples/test/resources/uvsphere.obj; visual mesh filename=package://exotica_examples/test/resources/uvsphere.obj

File: exotica_examples/test/resources/primitive_box_vs_mesh_distance.urdf (robot description, URDF)
Before this commit: robot A_vs_B, 2 links, 1 joints
Links:
- link A: geometry collision box size=2 2 2; visual box size=2 2 2
- link B: geometry collision mesh filename=package://exotica_examples/test/resources/uvsphere.obj; visual mesh filename=package://exotica_examples/test/resources/uvsphere.obj

File: exotica_examples/test/resources/primitive_box_vs_mesh_penetrating.urdf (robot description, URDF)
Before this commit: robot A_vs_B, 2 links, 1 joints
Links:
- link A: geometry collision box size=2 2 2; visual box size=2 2 2
- link B: geometry collision mesh filename=package://exotica_examples/test/resources/uvsphere.obj; visual mesh filename=package://exotica_examples/test/resources/uvsphere.obj

File: exotica_examples/test/resources/primitive_box_vs_primitive_box_distance.urdf (robot description, URDF)
Before this commit: robot A_vs_B, 2 links, 1 joints
Links:
- link A: geometry collision box size=1 1 1; visual box size=1 1 1
- link B: geometry collision box size=1 1 1; visual box size=1 1 1

File: exotica_examples/test/resources/primitive_box_vs_primitive_box_penetrating.urdf (robot description, URDF)
Before this commit: robot A_vs_B, 2 links, 1 joints
Links:
- link A: geometry collision box size=1 1 1; visual box size=1 1 1
- link B: geometry collision box size=1 1 1; visual box size=1 1 1

File: exotica_examples/test/resources/primitive_box_vs_primitive_box_touching.urdf (robot description, URDF)
Before this commit: robot A_vs_B, 2 links, 1 joints
Links:
- link A: geometry collision box size=1 1 1; visual box size=1 1 1
- link B: geometry collision box size=1 1 1; visual box size=1 1 1

File: exotica_examples/test/resources/primitive_box_vs_primitive_cylinder_distance.urdf (robot description, URDF)
Before this commit: robot A_vs_B, 2 links, 1 joints
Links:
- link A: geometry collision sphere radius=1; visual sphere radius=1
- link B: geometry collision cylinder length=1 radius=.25; visual cylinder length=1 radius=.25

File: exotica_examples/test/resources/primitive_box_vs_primitive_cylinder_penetrating.urdf (robot description, URDF)
Before this commit: robot A_vs_B, 2 links, 1 joints
Links:
- link A: geometry collision sphere radius=0.5; visual sphere radius=0.5
- link B: geometry collision cylinder length=1 radius=.25; visual cylinder length=1 radius=.25

File: exotica_examples/test/resources/primitive_cylinder_vs_mesh_distance.urdf (robot description, URDF)
Before this commit: robot A_vs_B, 2 links, 1 joints
Links:
- link A: geometry collision cylinder length=1 radius=.5; visual cylinder length=1 radius=.5
- link B: geometry collision mesh filename=package://exotica_examples/test/resources/uvsphere.obj; visual mesh filename=package://exotica_examples/test/resources/uvsphere.obj

File: exotica_examples/test/resources/primitive_cylinder_vs_mesh_penetrating.urdf (robot description, URDF)
Before this commit: robot A_vs_B, 2 links, 1 joints
Links:
- link A: geometry collision cylinder length=3 radius=.5; visual cylinder length=3 radius=.5
- link B: geometry collision mesh filename=package://exotica_examples/test/resources/uvsphere.obj; visual mesh filename=package://exotica_examples/test/resources/uvsphere.obj

File: exotica_examples/test/resources/primitive_cylinder_vs_primitive_cylinder_distance.urdf (robot description, URDF)
Before this commit: robot A_vs_B, 2 links, 1 joints
Links:
- link A: geometry collision cylinder length=1 radius=.5; visual cylinder length=1 radius=.5
- link B: geometry collision cylinder length=1 radius=.5; visual cylinder length=1 radius=.5

File: exotica_examples/test/resources/primitive_cylinder_vs_primitive_cylinder_penetrating.urdf (robot description, URDF)
Before this commit: robot A_vs_B, 2 links, 1 joints
Links:
- link A: geometry collision cylinder length=1 radius=.5; visual cylinder length=1 radius=.5
- link B: geometry collision cylinder length=1 radius=.5; visual cylinder length=1 radius=.5

File: exotica_examples/test/resources/primitive_sphere_vs_mesh_distance.urdf (robot description, URDF)
Before this commit: robot A_vs_B, 2 links, 1 joints
Links:
- link A: geometry collision sphere radius=1; visual sphere radius=1
- link B: geometry collision mesh filename=package://exotica_examples/test/resources/uvsphere.obj; visual mesh filename=package://exotica_examples/test/resources/uvsphere.obj

File: exotica_examples/test/resources/primitive_sphere_vs_mesh_penetrating.urdf (robot description, URDF)
Before this commit: robot A_vs_B, 2 links, 1 joints
Links:
- link A: geometry collision sphere radius=1; visual sphere radius=1
- link B: geometry collision mesh filename=package://exotica_examples/test/resources/uvsphere.obj; visual mesh filename=package://exotica_examples/test/resources/uvsphere.obj

File: exotica_examples/test/resources/primitive_sphere_vs_primitive_box_distance.urdf (robot description, URDF)
Before this commit: robot A_vs_B, 2 links, 1 joints
Links:
- link A: geometry collision sphere radius=1; visual sphere radius=1
- link B: geometry collision box size=1 1 1; visual box size=1 1 1

File: exotica_examples/test/resources/primitive_sphere_vs_primitive_box_penetrating.urdf (robot description, URDF)
Before this commit: robot A_vs_B, 2 links, 1 joints
Links:
- link A: geometry collision sphere radius=1; visual sphere radius=1
- link B: geometry collision box size=1 1 1; visual box size=1 1 1

File: exotica_examples/test/resources/primitive_sphere_vs_primitive_box_touching.urdf (robot description, URDF)
Before this commit: robot A_vs_B, 2 links, 1 joints
Links:
- link A: geometry collision sphere radius=1; visual sphere radius=1
- link B: geometry collision box size=1 1 1; visual box size=1 1 1
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